File: hardware/Double_Mos.kicad_sch (KiCad schematic)
At the start: 12 parts, among them U14 AOZ5276QI, U15 AOZ5276QI

Commit message: Revert "chore(schematic): Update references"
This reverts commit 2cda2d22061e90f93ddb38c43ecf32892cd7b43c.
Parts:
- renumbered C48 to C50, C49 to C51, C50 to C52, C51 to C53, C52 to C54, C53 to C55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

Commit message: chore(schematic): Update references
Parts:
- renumbered C50 to C48, C51 to C49, C52 to C50, C53 to C51, C54 to C52, C55 to C53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
