File: hardware/Onboard_Control.kicad_sch (KiCad schematic)
At the start: 6 parts, among them J8001 Conn_01x04_Pin, SW8001 CK_KMS2xxG, SW8002 CK_KMS2xxG, SW8003 CK_KMS2xxG, SW8004 CK_KMS2xxG, SW8005 CK_KMS2xxG

Commit message: chore: remove computer control and clean global references
Changed lines of the file:
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@@
-		)
-	)
-	(hierarchical_label "onbrd_cntrl_cntrllr_dsig"
-		(shape input)
-		(at 209.55 102.87 0)
-		(effects
-			(font
-				(size 1.27 1.27)
-			)
-			(justify left)
-		)
-	)
-	(hierarchical_label "otsd_onbrd_cntrl_usrin"
-		(shape input)
-		(at 229.87 107.95 180)
-		(effects
-			(font
-				(size 1.27 1.27)
-			)
-			(justify right)
 		)
 	)

Commit message: feat(schematic): added cooler mounting holes
added cooler mounting holes to schematic
changed temp pins to read proper tempurature
small fixes
Parts:
- SW8001, SW8002, SW8003, SW8004, SW8005: footprint work:SW_TS02-66-70-BK-160-LCR-D -> work:KEY-SMD_4P-L6.0-W6.0-P3.90-LS9.0
Changed lines of the file:
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@@
 			)
 		)
-		(property "Footprint" "work:SW_TS02-66-70-BK-160-LCR-D"
+		(property "Footprint" "work:KEY-SMD_4P-L6.0-W6.0-P3.90-LS9.0"
 			(at 36.83 102.87 0)
 			(effects
@@
 			)
 		)
-		(property "Datasheet" "https://www.ckswitches.com/media/1482/kms.pdf"
+		(property "Datasheet" "https://jlcpcb.com/partdetail/Korean_HropartsElec-K2_6639SP_C4SC04/C83206"
 			(at 36.83 102.87 0)
 			(effects
@@
 			)
 		)
-		(property "Footprint" "work:SW_TS02-66-70-BK-160-LCR-D"
+		(property "Footprint" "work:KEY-SMD_4P-L6.0-W6.0-P3.90-LS9.0"
 			(at 64.77 133.35 0)
 			(effects
@@
 			)
 		)
-		(property "Datasheet" "https://www.ckswitches.com/media/1482/kms.pdf"
+		(property "Datasheet" "https://jlcpcb.com/partdetail/Korean_HropartsElec-K2_6639SP_C4SC04/C83206"
 			(at 64.77 133.35 0)
 			(effects
@@
 			)
 		)
-		(property "Footprint" "work:SW_TS02-66-70-BK-160-LCR-D"
+		(property "Footprint" "work:KEY-SMD_4P-L6.0-W6.0-P3.90-LS9.0"
 			(at 91.44 102.87 0)
 			(effects
@@
 			)
 		)
-		(property "Datasheet" "https://www.ckswitches.com/media/1482/kms.pdf"
+		(property "Datasheet" "https://jlcpcb.com/partdetail/Korean_HropartsElec-K2_6639SP_C4SC04/C83206"
 			(at 91.44 102.87 0)
 			(effects
@@
 			)
 		)
-		(property "Footprint" "work:SW_TS02-66-70-BK-160-LCR-D"
+		(property "Footprint" "work:KEY-SMD_4P-L6.0-W6.0-P3.90-LS9.0"
 			(at 64.77 77.47 0)
 			(effects
@@
 			)
 		)
-		(property "Datasheet" "https://www.ckswitches.com/media/1482/kms.pdf"
+		(property "Datasheet" "https://jlcpcb.com/partdetail/Korean_HropartsElec-K2_6639SP_C4SC04/C83206"
 			(at 64.77 77.47 0)
 			(effects
@@
 			)
 		)
-		(property "Footprint" "work:SW_TS02-66-70-BK-160-LCR-D"
+		(property "Footprint" "work:KEY-SMD_4P-L6.0-W6.0-P3.90-LS9.0"
 			(at 64.77 105.41 0)
 			(effects
@@
 			)
 		)
-		(property "Datasheet" "https://www.digikey.com/en/products/detail/c-k/KMS223GP-LFG/679931"
+		(property "Datasheet" "https://jlcpcb.com/partdetail/Korean_HropartsElec-K2_6639SP_C4SC04/C83206"
 			(at 64.77 105.41 0)
 			(effects
@@
 			)
 		)
-		(property "Datasheet" "https://www.digikey.com/en/products/detail/sullins-connector-solutions/PPTC041LFBN-RC/810144"
+		(property "Datasheet" "https://jlcpcb.com/partdetail/125688-B_2200S04PA120/C124413"
 			(at 129.54 78.74 0)
 			(effects

Commit message: chore(schematic): add LCSC Part Numbers
Parts:
- J8001: LCSC Part Number (none) -> C124413
- SW8001, SW8002, SW8003, SW8004, SW8005: LCSC Part Number (none) -> C8326
Changed lines of the file:
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@@
+			)
+		)
+		(property "LCSC Part Number" "C8326"
+			(at 36.83 102.87 0)
+			(effects
+				(font
+					(size 1.27 1.27)
+				)
+				(hide yes)
 			)
 		)
@@
 			)
 		)
+		(property "LCSC Part Number" "C8326"
+			(at 64.77 133.35 0)
+			(effects
+				(font
+					(size 1.27 1.27)
+				)
+				(hide yes)
+			)
+		)
 		(pin "3"
 		)
@@
 				)
 				(justify bottom)
+				(hide yes)
+			)
+		)
+		(property "LCSC Part Number" "C8326"
+			(at 91.44 102.87 0)
+			(effects
+				(font
+					(size 1.27 1.27)
+				)
 				(hide yes)
 			)
@@
 			)
 		)
+		(property "LCSC Part Number" "C8326"
+			(at 64.77 77.47 0)
+			(effects
+				(font
+					(size 1.27 1.27)
+				)
+				(hide yes)
+			)
+		)
 		(pin "3"
 		)
@@
 				)
 				(justify bottom)
+				(hide yes)
+			)
+		)
+		(property "LCSC Part Number" "C8326"
+			(at 64.77 105.41 0)
+			(effects
+				(font
+					(size 1.27 1.27)
+				)
 				(hide yes)
 			)
@@
 			(at 129.54 78.74 0)
 			(effects
+				(font
+					(size 1.27 1.27)
+				)
+				(hide yes)
+			)
+		)
+		(property "LCSC Part Number" "C124413"
+			(at 129.54 78.74 0)
+			(effects
