File: hardware/12V_Supply.kicad_sch (KiCad schematic)
At the start: 27 parts, among them J1 Conn_01x06_Pin, J1 Conn_01x08_Pin, J2 Conn_01x06_Pin, J2 Conn_01x08_Pin, J3 Conn_01x06_Pin

Commit message: feat(schematic): Added Hall Sensor
Parts:
- removed D1 (x2), D2 (x2): D, symbol Device:D
- removed J1, J2: Conn_01x08_Pin, symbol Connector:Conn_01x08_Pin
- removed J1, J2, J3: Conn_01x06_Pin, symbol Connector:Conn_01x06_Pin
- added J1, J2, J3: 353180620, CONN_35318-06xx_MOL, symbol PCIe 2x3 Conn GPU:353180620
- added U17: ACS758xCB-150B-PSS, Sensor_Current:Allegro_CB_PSS, symbol Sensor_Current:ACS758xCB-150B-PSS
- renumbered C67 to C1, C71 to C3
Connections:
- net 12v_spply_lw_crrnt_spply_dcpwr: now also U17.5 (IP-); no longer C1.1, C3.1, C68.1, C69.1, C70.1, C72.1, L15.2, L16.2, L17.2
- net GND: now also C1.2, C3.2, C68.2, C69.2, C70.2, C72.2, J1.4, J1.6, J2.4, J2.6, J3.4, J3.6
- net Sense: now also J1.5, J2.5, J3.5
- net at C60.1, C63.1, C66.1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: now also J3.1, J3.2, J3.3
- net at C58.1, C61.1, C64.1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: now also J1.1, J1.2, J1.3
- net at C59.1, C62.1, C65.1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: now also J2.1, J2.2, J2.3
- new net: C1.1, C3.1, C68.1, C69.1, C70.1, C72.1, L15.2, L16.2, L17.2, U17.4 (IP+)

Commit message: chore: update project references
Parts:
- renumbered C58 to C4001, C59 to C4002, C60 to C4003, C61 to C4004, C62 to C4005, C63 to C4006, C64 to C4007, C65 to C4008, C66 to C4009, C68 to C4011, C69 to C4012, C70 to C4013, C72 to C4015, J1 to J4001, J2 to J4002, J3 to J4003, L15 to L4001, L16 to L4002, L17 to L4003, U17 to U4001
Changed lines of the file:
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@@
 			(project "gpu-external-power-supply"
 				(path "/d5303413-7068-41ba-88e3-39dfa38d31b7/c9569ad4-2b3d-43a2-87fb-13a0af7c9546"
-					(reference "C?")
+					(reference "C4010")
 					(unit 1)
 				)
@@
 		(dnp no)
 		(fields_autoplaced yes)
-		(property "Reference" "C66"
+		(property "Reference" "C4009"
 			(at 156.21 144.7799 0)
 			(effects
@@
 			(project "gpu-external-power-supply"
 				(path "/d5303413-7068-41ba-88e3-39dfa38d31b7/c9569ad4-2b3d-43a2-87fb-13a0af7c9546"
-					(reference "C66")
+					(reference "C4009")
 					(unit 1)
 				)
@@
 		(dnp no)
 		(fields_autoplaced yes)
-		(property "Reference" "C58"
+		(property "Reference" "C4001"
 			(at 125.73 50.7999 0)
 			(effects
@@
 			(project "gpu-external-power-supply"
 				(path "/d5303413-7068-41ba-88e3-39dfa38d31b7/c9569ad4-2b3d-43a2-87fb-13a0af7c9546"
-					(reference "C58")
+					(reference "C4001")
 					(unit 1)
 				)
@@
 		(dnp no)
 		(fields_autoplaced yes)
-		(property "Reference" "#PWR031"
+		(property "Reference" "#PWR04002"
 			(at 102.87 115.57 0)
 			(effects
@@
 			(project "gpu-external-power-supply"
 				(path "/d5303413-7068-41ba-88e3-39dfa38d31b7/c9569ad4-2b3d-43a2-87fb-13a0af7c9546"
-					(reference "#PWR031")
+					(reference "#PWR04002")
 					(unit 1)
 				)
@@
 		(on_board yes)
 		(dnp no)
-		(property "Reference" "U17"
+		(property "Reference" "U4001"
 			(at 234.696 70.866 90)
 			(effects
@@
 			(project ""
 				(path "/d5303413-7068-41ba-88e3-39dfa38d31b7/c9569ad4-2b3d-43a2-87fb-13a0af7c9546"
-					(reference "U17")
+					(reference "U4001")
 					(unit 1)
 				)
@@
 			(project "gpu-external-power-supply"
 				(path "/d5303413-7068-41ba-88e3-39dfa38d31b7/c9569ad4-2b3d-43a2-87fb-13a0af7c9546"
-					(reference "C?")
+					(reference "C4014")
 					(unit 1)
 				)
@@
 		(dnp no)
 		(fields_autoplaced yes)
-		(property "Reference" "C69"
+		(property "Reference" "C4012"
 			(at 180.34 144.7799 0)
 			(effects
@@
 			(project "gpu-external-power-supply"
 				(path "/d5303413-7068-41ba-88e3-39dfa38d31b7/c9569ad4-2b3d-43a2-87fb-13a0af7c9546"
-					(reference "C69")
+					(reference "C4012")
 					(unit 1)
 				)
@@
 		(dnp no)
 		(fields_autoplaced yes)
-		(property "Reference" "C63"
+		(property "Reference" "C4006"
 			(at 140.97 144.7799 0)
 			(effects
@@
 			(project "gpu-external-power-supply"
 				(path "/d5303413-7068-41ba-88e3-39dfa38d31b7/c9569ad4-2b3d-43a2-87fb-13a0af7c9546"
-					(reference "C63")
+					(reference "C4006")
 					(unit 1)
 				)
@@
 		(dnp no)
 		(fields_autoplaced yes)
-		(property "Reference" "C60"
+		(property "Reference" "C4003"
 			(at 125.73 144.7799 0)
 			(effects
@@
 			(project "gpu-external-power-supply"
 				(path "/d5303413-7068-41ba-88e3-39dfa38d31b7/c9569ad4-2b3d-43a2-87fb-13a0af7c9546"
-					(reference "C60")
+					(reference "C4003")
 					(unit 1)
 				)
@@
 			(project "gpu-external-power-supply"
 				(path "/d5303413-7068-41ba-88e3-39dfa38d31b7/c9569ad4-2b3d-43a2-87fb-13a0af7c9546"
-					(reference "#PWR?")
+					(reference "#PWR04003")
 					(unit 1)
 				)
@@
 		(dnp no)
 		(fields_autoplaced yes)
-		(property "Reference" "C64"
+		(property "Reference" "C4007"
 			(at 156.21 50.7999 0)
 			(effects
@@
 			(project "gpu-external-power-supply"
 				(path "/d5303413-7068-41ba-88e3-39dfa38d31b7/c9569ad4-2b3d-43a2-87fb-13a0af7c9546"
-					(reference "C64")
+					(reference "C4007")
 					(unit 1)
 				)
@@
 		(dnp no)
 		(fields_autoplaced yes)
-		(property "Reference" "C65"
+		(property "Reference" "C4008"
 			(at 156.21 97.7899 0)
 			(effects
@@
 			(project "gpu-external-power-supply"
 				(path "/d5303413-7068-41ba-88e3-39dfa38d31b7/c9569ad4-2b3d-43a2-87fb-13a0af7c9546"
-					(reference "C65")
+					(reference "C4008")
 					(unit 1)
 				)
@@
 			(project "gpu-external-power-supply"
 				(path "/d5303413-7068-41ba-88e3-39dfa38d31b7/c9569ad4-2b3d-43a2-87fb-13a0af7c9546"
-					(reference "#PWR?")
+					(reference "#PWR04004")
 					(unit 1)
 				)
@@
 		(dnp no)
 		(fields_autoplaced yes)
-		(property "Reference" "C70"
+		(property "Reference" "C4013"
 			(at 196.85 50.7999 0)
 			(effects
@@
 			(project "gpu-external-power-supply"
 				(path "/d5303413-7068-41ba-88e3-39dfa38d31b7/c9569ad4-2b3d-43a2-87fb-13a0af7c9546"
-					(reference "C70")
+					(reference "C4013")
 					(unit 1)
 				)
@@
 		(dnp no)
 		(fields_autoplaced yes)
-		(property "Reference" "L17"
+		(property "Reference" "L4003"
 			(at 163.83 134.62 90)
 			(effects
@@
 			(project "gpu-external-power-supply"
 				(path "/d5303413-7068-41ba-88e3-39dfa38d31b7/c9569ad4-2b3d-43a2-87fb-13a0af7c9546"
-					(reference "L17")
+					(reference "L4003")
 					(unit 1)
 				)
@@
 		(dnp no)
 		(fields_autoplaced yes)
-		(property "Reference" "C72"
+		(property "Reference" "C4015"
 			(at 196.85 144.7799 0)
 			(effects
@@
 			(project "gpu-external-power-supply"
 				(path "/d5303413-7068-41ba-88e3-39dfa38d31b7/c9569ad4-2b3d-43a2-87fb-13a0af7c9546"
-					(reference "C72")
+					(reference "C4015")
 					(unit 1)
 				)
@@
 		(dnp no)
 		(fields_autoplaced yes)
-		(property "Reference" "#PWR032"
+		(property "Reference" "#PWR04006"
 			(at 176.53 157.48 0)
 			(effects
@@
 			(project "gpu-external-power-supply"
 				(path "/d5303413-7068-41ba-88e3-39dfa38d31b7/c9569ad4-2b3d-43a2-87fb-13a0af7c9546"
-					(reference "#PWR032")
+					(reference "#PWR04006")
 					(unit 1)
 				)
@@
 		(dnp no)
 		(fields_autoplaced yes)
-		(property "Reference" "J3"
+		(property "Reference" "J4003"
 			(at 71.12 121.92 0)
 			(effects
@@
 			(project "gpu-external-power-supply"
 				(path "/d5303413-7068-41ba-88e3-39dfa38d31b7/c9569ad4-2b3d-43a2-87fb-13a0af7c9546"
-					(reference "J3")
+					(reference "J4003")
 					(unit 1)
 				)
@@
 		(dnp no)
 		(fields_autoplaced yes)
-		(property "Reference" "C68"
+		(property "Reference" "C4011"
 			(at 180.34 97.7899 0)
 			(effects
@@
 			(project "gpu-external-power-supply"
 				(path "/d5303413-7068-41ba-88e3-39dfa38d31b7/c9569ad4-2b3d-43a2-87fb-13a0af7c9546"
-					(reference "C68")
+					(reference "C4011")
 					(unit 1)
 				)
@@
 		(dnp no)
 		(fields_autoplaced yes)
-		(property "Reference" "L15"
+		(property "Reference" "L4001"
 			(at 163.83 40.64 90)
 			(effects
@@
 			(project "gpu-external-power-supply"
 				(path "/d5303413-7068-41ba-88e3-39dfa38d31b7/c9569ad4-2b3d-43a2-87fb-13a0af7c9546"
-					(reference "L15")
+					(reference "L4001")
 					(unit 1)
 				)
@@
 		(dnp no)
 		(fields_autoplaced yes)
-		(property "Reference" "C61"
+		(property "Reference" "C4004"
 			(at 140.97 50.7999 0)
 			(effects
@@
 			(project "gpu-external-power-supply"
 				(path "/d5303413-7068-41ba-88e3-39dfa38d31b7/c9569ad4-2b3d-43a2-87fb-13a0af7c9546"
-					(reference "C61")
+					(reference "C4004")
 					(unit 1)
 				)
@@
 		(dnp no)
 		(fields_autoplaced yes)
-		(property "Reference" "J1"
+		(property "Reference" "J4001"
 			(at 71.12 25.4 0)
 			(effects
@@
 			(project "gpu-external-power-supply"
 				(path "/d5303413-7068-41ba-88e3-39dfa38d31b7/c9569ad4-2b3d-43a2-87fb-13a0af7c9546"
-					(reference "J1")
+					(reference "J4001")
 					(unit 1)
 				)
@@
 		(dnp no)
 		(fields_autoplaced yes)
-		(property "Reference" "C62"
+		(property "Reference" "C4005"
 			(at 140.97 97.7899 0)
 			(effects
@@
 			(project "gpu-external-power-supply"
 				(path "/d5303413-7068-41ba-88e3-39dfa38d31b7/c9569ad4-2b3d-43a2-87fb-13a0af7c9546"
-					(reference "C62")
+					(reference "C4005")
 					(unit 1)
 				)
@@
 		(dnp no)
 		(fields_autoplaced yes)
-		(property "Reference" "#PWR030"
+		(property "Reference" "#PWR04001"
 			(at 102.87 68.58 0)
 			(effects
@@
 			(project "gpu-external-power-supply"
 				(path "/d5303413-7068-41ba-88e3-39dfa38d31b7/c9569ad4-2b3d-43a2-87fb-13a0af7c9546"
-					(reference "#PWR030")
+					(reference "#PWR04001")
 					(unit 1)
 				)
@@
 		(dnp no)
 		(fields_autoplaced yes)
-		(property "Reference" "L16"
+		(property "Reference" "L4002"
 			(at 163.83 87.63 90)
 			(effects
@@
 			(project "gpu-external-power-supply"
 				(path "/d5303413-7068-41ba-88e3-39dfa38d31b7/c9569ad4-2b3d-43a2-87fb-13a0af7c9546"
-					(reference "L16")
+					(reference "L4002")
 					(unit 1)
 				)
@@
 		(dnp no)
 		(fields_autoplaced yes)
-		(property "Reference" "C59"
+		(property "Reference" "C4002"
 			(at 125.73 97.7899 0)
 			(effects
@@
 			(project "gpu-external-power-supply"
 				(path "/d5303413-7068-41ba-88e3-39dfa38d31b7/c9569ad4-2b3d-43a2-87fb-13a0af7c9546"
-					(reference "C59")
+					(reference "C4002")
 					(unit 1)
 				)
@@
 			(project "gpu-external-power-supply"
 				(path "/d5303413-7068-41ba-88e3-39dfa38d31b7/c9569ad4-2b3d-43a2-87fb-13a0af7c9546"
-					(reference "#PWR?")
+					(reference "#PWR04005")
 					(unit 1)
 				)
@@
 		(dnp no)
 		(fields_autoplaced yes)
-		(property "Reference" "J2"
+		(property "Reference" "J4002"
 			(at 71.12 72.39 0)
 			(effects
@@
 			(project "gpu-external-power-supply"
 				(path "/d5303413-7068-41ba-88e3-39dfa38d31b7/c9569ad4-2b3d-43a2-87fb-13a0af7c9546"
-					(reference "J2")
-					(unit 1)
-				)
+					(reference "J4002")
+					(unit 1)
+				)
