File: hardware/gpu-external-power-supply.kicad_pcb (KiCad board)
At the start: 6 copper layers, 170.2 x 99.1 mm, 101 parts, among them J4001 353180620, J4002 353180620, J4004 353180620, J7002 Conn_ARM_JTAG_SWD_10, J7003 USB_C_Receptacle_USB2.0_16P, J8001 Conn_01x04_Pin, SW7001 SW_Wuerth_450301014042, SW8001 CK_KMS2xxG, SW8002 CK_KMS2xxG, SW8003 CK_KMS2xxG, SW8004 CK_KMS2xxG, SW8005 CK_KMS2xxG, U5001 TPS62160DSG, U5002 TPS73633DBVR, U7002 STM32C071RBT6, U7003 USBLC6-2SC6, Y7001 Crystal_GND24

Commit message: feat(PCB): low-current-supply layout
Parts:
- removed R5, R6, R7, R8: 0, Resistor_SMD:R_2512_6332Metric_Pad1.40x3.35mm_HandSolder
- added C11001: 47pF, Capacitor_SMD:C_0805_2012Metric, F.Cu at (393.4, 203.6)
- added C11002: 2.2uF, Capacitor_SMD:C_0805_2012Metric, F.Cu at (393.4, 206.6)
- added C11003: 0.1uF, Capacitor_SMD:C_0805_2012Metric, F.Cu at (393.4, 209.6)
- added C11004: 2.2uF, Capacitor_SMD:C_0805_2012Metric, F.Cu at (393.4, 212.7)
- added C11005: 47pF, Capacitor_SMD:C_0805_2012Metric, F.Cu at (393.4, 215.7)
- added C11006: 0.1uF, Capacitor_SMD:C_0805_2012Metric, F.Cu at (397.8, 203.6)
- added C11007: 0.1uF, Capacitor_SMD:C_0805_2012Metric, F.Cu at (397.8, 206.6)
- added C11008: 22uF, Capacitor_SMD:C_0805_2012Metric, F.Cu at (397.8, 209.6)
- added C11009: 470uF, work:CP_EIA-7343-40_Kemet-Y, F.Cu at (409.5, 205.0)
- added C11010: 22uF, Capacitor_SMD:C_0805_2012Metric, F.Cu at (397.8, 212.7)
- added C11011: 220uF, Capacitor_THT:CP_Radial_D6.3mm_P2.50mm, F.Cu at (407.3, 211.9)
- added C11012: 22uF, Capacitor_SMD:C_0805_2012Metric, F.Cu at (397.8, 215.7)
- added C11013: 47uF, Capacitor_SMD:C_0805_2012Metric, F.Cu at (402.3, 203.6)
- added C11014: 220uF, Capacitor_THT:CP_Radial_D6.3mm_P2.50mm, F.Cu at (407.3, 219.7)
- added C11015: 22uF, Capacitor_SMD:C_0805_2012Metric, F.Cu at (402.3, 206.6)
- added C11016: 4.7uF, Capacitor_SMD:C_0805_2012Metric, F.Cu at (402.3, 209.6)
- added C11017: 0.1uF, Capacitor_SMD:C_0805_2012Metric, F.Cu at (402.3, 212.7)
- added C12001: 47pF, Capacitor_SMD:C_0805_2012Metric, F.Cu at (333.9, 203.6)
- added C12002: 2.2uF, Capacitor_SMD:C_0805_2012Metric, F.Cu at (333.9, 206.6)
- added C12003: 0.1uF, Capacitor_SMD:C_0805_2012Metric, F.Cu at (333.9, 209.6)
- added C12004: 2.2uF, Capacitor_SMD:C_0805_2012Metric, F.Cu at (333.9, 212.7)
- added C12005: 47pF, Capacitor_SMD:C_0805_2012Metric, F.Cu at (333.9, 215.7)
- added C12006: 0.1uF, Capacitor_SMD:C_0805_2012Metric, F.Cu at (338.4, 203.6)
- added C12007: 0.1uF, Capacitor_SMD:C_0805_2012Metric, F.Cu at (338.4, 206.6)
- added C12008: 22uF, Capacitor_SMD:C_0805_2012Metric, F.Cu at (338.4, 209.6)
- added C12009: 470uF, work:CP_EIA-7343-40_Kemet-Y, F.Cu at (350.0, 205.0)
- added C12010: 22uF, Capacitor_SMD:C_0805_2012Metric, F.Cu at (338.4, 212.7)
- added C12011: 220uF, Capacitor_THT:CP_Radial_D6.3mm_P2.50mm, F.Cu at (347.9, 211.9)
- added C12012: 22uF, Capacitor_SMD:C_0805_2012Metric, F.Cu at (338.4, 215.7)
- added C12013: 47uF, Capacitor_SMD:C_0805_2012Metric, F.Cu at (342.8, 203.6)
- added C12014: 220uF, Capacitor_THT:CP_Radial_D6.3mm_P2.50mm, F.Cu at (347.9, 219.7)
- added C12015: 22uF, Capacitor_SMD:C_0805_2012Metric, F.Cu at (342.8, 206.6)
- added C12016: 4.7uF, Capacitor_SMD:C_0805_2012Metric, F.Cu at (342.8, 209.6)
- added C12017: 0.1uF, Capacitor_SMD:C_0805_2012Metric, F.Cu at (342.8, 212.7)
- added C13001: 47pF, Capacitor_SMD:C_0805_2012Metric, F.Cu at (363.6, 203.6)
- added C13002: 2.2uF, Capacitor_SMD:C_0805_2012Metric, F.Cu at (363.6, 206.6)
- added C13003: 0.1uF, Capacitor_SMD:C_0805_2012Metric, F.Cu at (363.6, 209.6)
- added C13004: 2.2uF, Capacitor_SMD:C_0805_2012Metric, F.Cu at (363.6, 212.7)
- added C13005: 47pF, Capacitor_SMD:C_0805_2012Metric, F.Cu at (363.6, 215.7)
- added C13006: 0.1uF, Capacitor_SMD:C_0805_2012Metric, F.Cu at (368.1, 203.6)
- added C13007: 0.1uF, Capacitor_SMD:C_0805_2012Metric, F.Cu at (368.1, 206.6)
- added C13008: 22uF, Capacitor_SMD:C_0805_2012Metric, F.Cu at (368.1, 209.6)
- added C13009: 470uF, work:CP_EIA-7343-40_Kemet-Y, F.Cu at (379.7, 205.0)
- added C13010: 22uF, Capacitor_SMD:C_0805_2012Metric, F.Cu at (368.1, 212.7)
- added C13011: 220uF, Capacitor_THT:CP_Radial_D6.3mm_P2.50mm, F.Cu at (377.6, 211.9)
- added C13012: 22uF, Capacitor_SMD:C_0805_2012Metric, F.Cu at (368.1, 215.7)
- added C13013: 47uF, Capacitor_SMD:C_0805_2012Metric, F.Cu at (372.5, 203.6)
- added C13014: 220uF, Capacitor_THT:CP_Radial_D6.3mm_P2.50mm, F.Cu at (377.6, 219.7)
- added C13015: 22uF, Capacitor_SMD:C_0805_2012Metric, F.Cu at (372.5, 206.6)
- added C13016: 4.7uF, Capacitor_SMD:C_0805_2012Metric, F.Cu at (372.5, 209.6)
- added C13017: 0.1uF, Capacitor_SMD:C_0805_2012Metric, F.Cu at (372.5, 212.7)
- added C14001: 47pF, Capacitor_SMD:C_0805_2012Metric, F.Cu at (363.6, 253.8)
- added C14002: 2.2uF, Capacitor_SMD:C_0805_2012Metric, F.Cu at (363.6, 256.9)
- added C14003: 0.1uF, Capacitor_SMD:C_0805_2012Metric, F.Cu at (363.6, 259.9)
- added C14004: 2.2uF, Capacitor_SMD:C_0805_2012Metric, F.Cu at (363.6, 262.9)
- added C14005: 47pF, Capacitor_SMD:C_0805_2012Metric, F.Cu at (363.6, 265.9)
- added C14006: 0.1uF, Capacitor_SMD:C_0805_2012Metric, F.Cu at (368.1, 253.8)
- added C14007: 0.1uF, Capacitor_SMD:C_0805_2012Metric, F.Cu at (368.1, 256.9)
- added C14008: 22uF, Capacitor_SMD:C_0805_2012Metric, F.Cu at (368.1, 259.9)
- added C14009: 470uF, work:CP_EIA-7343-40_Kemet-Y, F.Cu at (379.7, 255.3)
- added C14010: 22uF, Capacitor_SMD:C_0805_2012Metric, F.Cu at (368.1, 262.9)
- added C14011: 220uF, Capacitor_THT:CP_Radial_D6.3mm_P2.50mm, F.Cu at (377.6, 262.1)
- added C14012: 22uF, Capacitor_SMD:C_0805_2012Metric, F.Cu at (368.1, 265.9)
- added C14013: 47uF, Capacitor_SMD:C_0805_2012Metric, F.Cu at (372.5, 253.8)
- added C14014: 220uF, Capacitor_THT:CP_Radial_D6.3mm_P2.50mm, F.Cu at (377.6, 270.0)
- added C14015: 22uF, Capacitor_SMD:C_0805_2012Metric, F.Cu at (372.5, 256.9)
- added C14016: 4.7uF, Capacitor_SMD:C_0805_2012Metric, F.Cu at (372.5, 259.9)
- added C14017: 0.1uF, Capacitor_SMD:C_0805_2012Metric, F.Cu at (372.5, 262.9)
- added C15001: 47pF, Capacitor_SMD:C_0805_2012Metric, F.Cu at (333.9, 228.7)
- added C15002: 2.2uF, Capacitor_SMD:C_0805_2012Metric, F.Cu at (333.9, 231.7)
- added C15003: 0.1uF, Capacitor_SMD:C_0805_2012Metric, F.Cu at (333.9, 234.8)
- added C15004: 2.2uF, Capacitor_SMD:C_0805_2012Metric, F.Cu at (333.9, 237.8)
- added C15005: 47pF, Capacitor_SMD:C_0805_2012Metric, F.Cu at (333.9, 240.8)
- added C15006: 0.1uF, Capacitor_SMD:C_0805_2012Metric, F.Cu at (338.4, 228.7)
- added C15007: 0.1uF, Capacitor_SMD:C_0805_2012Metric, F.Cu at (338.4, 231.7)
- added C15008: 22uF, Capacitor_SMD:C_0805_2012Metric, F.Cu at (338.4, 234.8)
- added C15009: 470uF, work:CP_EIA-7343-40_Kemet-Y, F.Cu at (350.0, 230.2)
- added C15010: 22uF, Capacitor_SMD:C_0805_2012Metric, F.Cu at (338.4, 237.8)
- added C15011: 220uF, Capacitor_THT:CP_Radial_D6.3mm_P2.50mm, F.Cu at (347.9, 237.0)
- added C15012: 22uF, Capacitor_SMD:C_0805_2012Metric, F.Cu at (338.4, 240.8)
- added C15013: 47uF, Capacitor_SMD:C_0805_2012Metric, F.Cu at (342.8, 228.7)
- added C15014: 220uF, Capacitor_THT:CP_Radial_D6.3mm_P2.50mm, F.Cu at (347.9, 244.8)
- added C15015: 22uF, Capacitor_SMD:C_0805_2012Metric, F.Cu at (342.8, 231.7)
- added C15016: 4.7uF, Capacitor_SMD:C_0805_2012Metric, F.Cu at (342.8, 234.8)
- added C15017: 0.1uF, Capacitor_SMD:C_0805_2012Metric, F.Cu at (342.8, 237.8)
- added C16018: 47pF, Capacitor_SMD:C_0805_2012Metric, F.Cu at (333.9, 178.5)
- added C16019: 2.2uF, Capacitor_SMD:C_0805_2012Metric, F.Cu at (333.9, 181.5)
- added C16020: 0.1uF, Capacitor_SMD:C_0805_2012Metric, F.Cu at (333.9, 184.5)
- added C16021: 2.2uF, Capacitor_SMD:C_0805_2012Metric, F.Cu at (333.9, 187.5)
- added C16022: 47pF, Capacitor_SMD:C_0805_2012Metric, F.Cu at (333.9, 190.6)
- added C16023: 0.1uF, Capacitor_SMD:C_0805_2012Metric, F.Cu at (338.4, 178.5)
- added C16024: 0.1uF, Capacitor_SMD:C_0805_2012Metric, F.Cu at (338.4, 181.5)
- added C16025: 22uF, Capacitor_SMD:C_0805_2012Metric, F.Cu at (338.4, 184.5)
- added C16026: 470uF, work:CP_EIA-7343-40_Kemet-Y, F.Cu at (350.0, 179.9)
- added C16027: 22uF, Capacitor_SMD:C_0805_2012Metric, F.Cu at (338.4, 187.5)
- added C16028: 220uF, Capacitor_THT:CP_Radial_D6.3mm_P2.50mm, F.Cu at (347.9, 186.8)
- added C16029: 22uF, Capacitor_SMD:C_0805_2012Metric, F.Cu at (338.4, 190.6)
- added C16030: 47uF, Capacitor_SMD:C_0805_2012Metric, F.Cu at (342.8, 178.5)
- added C16031: 220uF, Capacitor_THT:CP_Radial_D6.3mm_P2.50mm, F.Cu at (347.9, 194.6)
- added C16032: 22uF, Capacitor_SMD:C_0805_2012Metric, F.Cu at (342.8, 181.5)
- added C16033: 4.7uF, Capacitor_SMD:C_0805_2012Metric, F.Cu at (342.8, 184.5)
- added C16034: 0.1uF, Capacitor_SMD:C_0805_2012Metric, F.Cu at (342.8, 187.5)
- added C17001: 47pF, Capacitor_SMD:C_0805_2012Metric, F.Cu at (393.4, 228.7)
- added C17002: 2.2uF, Capacitor_SMD:C_0805_2012Metric, F.Cu at (393.4, 231.7)
- added C17003: 0.1uF, Capacitor_SMD:C_0805_2012Metric, F.Cu at (393.4, 234.8)
- added C17004: 2.2uF, Capacitor_SMD:C_0805_2012Metric, F.Cu at (393.4, 237.8)
- added C17005: 47pF, Capacitor_SMD:C_0805_2012Metric, F.Cu at (393.4, 240.8)
- added C17006: 0.1uF, Capacitor_SMD:C_0805_2012Metric, F.Cu at (397.8, 228.7)
- added C17007: 0.1uF, Capacitor_SMD:C_0805_2012Metric, F.Cu at (397.8, 231.7)
- added C17008: 22uF, Capacitor_SMD:C_0805_2012Metric, F.Cu at (397.8, 234.8)
- added C17009: 470uF, work:CP_EIA-7343-40_Kemet-Y, F.Cu at (409.5, 230.2)
- added C17010: 22uF, Capacitor_SMD:C_0805_2012Metric, F.Cu at (397.8, 237.8)
- added C17011: 220uF, Capacitor_THT:CP_Radial_D6.3mm_P2.50mm, F.Cu at (407.3, 237.0)
- added C17012: 22uF, Capacitor_SMD:C_0805_2012Metric, F.Cu at (397.8, 240.8)
- added C17013: 47uF, Capacitor_SMD:C_0805_2012Metric, F.Cu at (402.3, 228.7)
- added C17014: 220uF, Capacitor_THT:CP_Radial_D6.3mm_P2.50mm, F.Cu at (407.3, 244.8)
- added C17015: 22uF, Capacitor_SMD:C_0805_2012Metric, F.Cu at (402.3, 231.7)
- added C17016: 4.7uF, Capacitor_SMD:C_0805_2012Metric, F.Cu at (402.3, 234.8)
- added C17017: 0.1uF, Capacitor_SMD:C_0805_2012Metric, F.Cu at (402.3, 237.8)
- added C18001: 47pF, Capacitor_SMD:C_0805_2012Metric, F.Cu at (363.6, 178.5)
- added C18002: 2.2uF, Capacitor_SMD:C_0805_2012Metric, F.Cu at (363.6, 181.5)
- added C18003: 0.1uF, Capacitor_SMD:C_0805_2012Metric, F.Cu at (363.6, 184.5)
- added C18004: 2.2uF, Capacitor_SMD:C_0805_2012Metric, F.Cu at (363.6, 187.5)
- added C18005: 47pF, Capacitor_SMD:C_0805_2012Metric, F.Cu at (363.6, 190.6)
- added C18006: 0.1uF, Capacitor_SMD:C_0805_2012Metric, F.Cu at (368.1, 178.5)
- added C18007: 0.1uF, Capacitor_SMD:C_0805_2012Metric, F.Cu at (368.1, 181.5)
- added C18008: 22uF, Capacitor_SMD:C_0805_2012Metric, F.Cu at (368.1, 184.5)
- added C18009: 470uF, work:CP_EIA-7343-40_Kemet-Y, F.Cu at (379.7, 179.9)
- added C18010: 22uF, Capacitor_SMD:C_0805_2012Metric, F.Cu at (368.1, 187.5)
- added C18011: 220uF, Capacitor_THT:CP_Radial_D6.3mm_P2.50mm, F.Cu at (377.6, 186.8)
- added C18012: 22uF, Capacitor_SMD:C_0805_2012Metric, F.Cu at (368.1, 190.6)
- added C18013: 47uF, Capacitor_SMD:C_0805_2012Metric, F.Cu at (372.5, 178.5)
- added C18014: 220uF, Capacitor_THT:CP_Radial_D6.3mm_P2.50mm, F.Cu at (377.6, 194.6)
- added C18015: 22uF, Capacitor_SMD:C_0805_2012Metric, F.Cu at (372.5, 181.5)
- added C18016: 4.7uF, Capacitor_SMD:C_0805_2012Metric, F.Cu at (372.5, 184.5)
- added C18017: 0.1uF, Capacitor_SMD:C_0805_2012Metric, F.Cu at (372.5, 187.5)
- added C19001: 47pF, Capacitor_SMD:C_0805_2012Metric, F.Cu at (333.9, 253.8)
- added C19002: 2.2uF, Capacitor_SMD:C_0805_2012Metric, F.Cu at (333.9, 256.9)
- added C19003: 0.1uF, Capacitor_SMD:C_0805_2012Metric, F.Cu at (333.9, 259.9)
- added C19004: 2.2uF, Capacitor_SMD:C_0805_2012Metric, F.Cu at (333.9, 262.9)
- added C19005: 47pF, Capacitor_SMD:C_0805_2012Metric, F.Cu at (333.9, 265.9)
- added C19006: 0.1uF, Capacitor_SMD:C_0805_2012Metric, F.Cu at (338.4, 253.8)
- added C19007: 0.1uF, Capacitor_SMD:C_0805_2012Metric, F.Cu at (338.4, 256.9)
- added C19008: 22uF, Capacitor_SMD:C_0805_2012Metric, F.Cu at (338.4, 259.9)
- added C19009: 470uF, work:CP_EIA-7343-40_Kemet-Y, F.Cu at (350.0, 255.3)
- added C19010: 22uF, Capacitor_SMD:C_0805_2012Metric, F.Cu at (338.4, 262.9)
- added C19011: 220uF, Capacitor_THT:CP_Radial_D6.3mm_P2.50mm, F.Cu at (347.9, 262.1)
- added C19012: 22uF, Capacitor_SMD:C_0805_2012Metric, F.Cu at (338.4, 265.9)
- added C19013: 47uF, Capacitor_SMD:C_0805_2012Metric, F.Cu at (342.8, 253.8)
- added C19014: 220uF, Capacitor_THT:CP_Radial_D6.3mm_P2.50mm, F.Cu at (347.9, 270.0)
- added C19015: 22uF, Capacitor_SMD:C_0805_2012Metric, F.Cu at (342.8, 256.9)
- added C19016: 4.7uF, Capacitor_SMD:C_0805_2012Metric, F.Cu at (342.8, 259.9)
- added C19017: 0.1uF, Capacitor_SMD:C_0805_2012Metric, F.Cu at (342.8, 262.9)
- added C3001: 47pF, Capacitor_SMD:C_0805_2012Metric, F.Cu at (393.4, 178.5)
- added C3002: 2.2uF, Capacitor_SMD:C_0805_2012Metric, F.Cu at (393.4, 181.5)
- added C3003: 0.1uF, Capacitor_SMD:C_0805_2012Metric, F.Cu at (393.4, 184.5)
- added C3004: 2.2uF, Capacitor_SMD:C_0805_2012Metric, F.Cu at (393.4, 187.5)
- added C3005: 47pF, Capacitor_SMD:C_0805_2012Metric, F.Cu at (393.4, 190.6)
- added C3006: 0.1uF, Capacitor_SMD:C_0805_2012Metric, F.Cu at (397.8, 178.5)
- added C3007: 0.1uF, Capacitor_SMD:C_0805_2012Metric, F.Cu at (397.8, 181.5)
- added C3008: 22uF, Capacitor_SMD:C_0805_2012Metric, F.Cu at (397.8, 184.5)
- added C3009: 470uF, work:CP_EIA-7343-40_Kemet-Y, F.Cu at (409.5, 179.9)
- added C3010: 22uF, Capacitor_SMD:C_0805_2012Metric, F.Cu at (397.8, 187.5)
- added C3011: 220uF, Capacitor_THT:CP_Radial_D6.3mm_P2.50mm, F.Cu at (407.3, 186.8)
- added C3012: 22uF, Capacitor_SMD:C_0805_2012Metric, F.Cu at (397.8, 190.6)
- added C3013: 47uF, Capacitor_SMD:C_0805_2012Metric, F.Cu at (402.3, 178.5)
- added C3014: 220uF, Capacitor_THT:CP_Radial_D6.3mm_P2.50mm, F.Cu at (407.3, 194.6)
- added C3015: 22uF, Capacitor_SMD:C_0805_2012Metric, F.Cu at (402.3, 181.5)
- added C3016: 4.7uF, Capacitor_SMD:C_0805_2012Metric, F.Cu at (402.3, 184.5)
- added C3017: 0.1uF, Capacitor_SMD:C_0805_2012Metric, F.Cu at (402.3, 187.5)
- added C6001: 47pF, Capacitor_SMD:C_0805_2012Metric, F.Cu at (393.4, 253.8)
- added C6002: 2.2uF, Capacitor_SMD:C_0805_2012Metric, F.Cu at (393.4, 256.9)
- added C6003: 0.1uF, Capacitor_SMD:C_0805_2012Metric, F.Cu at (393.4, 259.9)
- added C6004: 2.2uF, Capacitor_SMD:C_0805_2012Metric, F.Cu at (393.4, 262.9)
- added C6005: 47pF, Capacitor_SMD:C_0805_2012Metric, F.Cu at (393.4, 265.9)
- added C6006: 0.1uF, Capacitor_SMD:C_0805_2012Metric, F.Cu at (397.8, 253.8)
- added C6007: 0.1uF, Capacitor_SMD:C_0805_2012Metric, F.Cu at (397.8, 256.9)
- added C6008: 22uF, Capacitor_SMD:C_0805_2012Metric, F.Cu at (397.8, 259.9)
- added C6009: 470uF, work:CP_EIA-7343-40_Kemet-Y, F.Cu at (409.5, 255.3)
- added C6010: 22uF, Capacitor_SMD:C_0805_2012Metric, F.Cu at (397.8, 262.9)
- added C6011: 220uF, Capacitor_THT:CP_Radial_D6.3mm_P2.50mm, F.Cu at (407.3, 262.1)
- added C6012: 22uF, Capacitor_SMD:C_0805_2012Metric, F.Cu at (397.8, 265.9)
- added C6013: 47uF, Capacitor_SMD:C_0805_2012Metric, F.Cu at (402.3, 253.8)
- added C6014: 220uF, Capacitor_THT:CP_Radial_D6.3mm_P2.50mm, F.Cu at (407.3, 270.0)
- added C6015: 22uF, Capacitor_SMD:C_0805_2012Metric, F.Cu at (402.3, 256.9)
- added C6016: 4.7uF, Capacitor_SMD:C_0805_2012Metric, F.Cu at (402.3, 259.9)
- added C6017: 0.1uF, Capacitor_SMD:C_0805_2012Metric, F.Cu at (402.3, 262.9)
- added C9001: 47pF, Capacitor_SMD:C_0805_2012Metric, F.Cu at (363.6, 228.7)
- added C9002: 2.2uF, Capacitor_SMD:C_0805_2012Metric, F.Cu at (363.6, 231.7)
- added C9003: 0.1uF, Capacitor_SMD:C_0805_2012Metric, F.Cu at (363.6, 234.8)
- added C9004: 2.2uF, Capacitor_SMD:C_0805_2012Metric, F.Cu at (363.6, 237.8)
- added C9005: 47pF, Capacitor_SMD:C_0805_2012Metric, F.Cu at (363.6, 240.8)
- added C9006: 0.1uF, Capacitor_SMD:C_0805_2012Metric, F.Cu at (368.1, 228.7)
- added C9007: 0.1uF, Capacitor_SMD:C_0805_2012Metric, F.Cu at (368.1, 231.7)
- added C9008: 22uF, Capacitor_SMD:C_0805_2012Metric, F.Cu at (368.1, 234.8)
- added C9009: 470uF, work:CP_EIA-7343-40_Kemet-Y, F.Cu at (379.7, 230.2)
- added C9010: 22uF, Capacitor_SMD:C_0805_2012Metric, F.Cu at (368.1, 237.8)
- added C9011: 220uF, Capacitor_THT:CP_Radial_D6.3mm_P2.50mm, F.Cu at (377.6, 237.0)
- added C9012: 22uF, Capacitor_SMD:C_0805_2012Metric, F.Cu at (368.1, 240.8)
- added C9013: 47uF, Capacitor_SMD:C_0805_2012Metric, F.Cu at (372.5, 228.7)
- added C9014: 220uF, Capacitor_THT:CP_Radial_D6.3mm_P2.50mm, F.Cu at (377.6, 244.8)
- added C9015: 22uF, Capacitor_SMD:C_0805_2012Metric, F.Cu at (372.5, 231.7)
- added C9016: 4.7uF, Capacitor_SMD:C_0805_2012Metric, F.Cu at (372.5, 234.8)
- added C9017: 0.1uF, Capacitor_SMD:C_0805_2012Metric, F.Cu at (372.5, 237.8)
- added J2001: Conn_01x02_Pin, Connector_PinHeader_2.54mm:PinHeader_1x02_P2.54mm_Vertical, F.Cu at (423.2, 254.7)
- added J2002: Conn_01x02_Pin, Connector_PinHeader_2.54mm:PinHeader_1x02_P2.54mm_Vertical, F.Cu at (427.9, 254.7)
- added J2003: Conn_01x02_Pin, Connector_PinHeader_2.54mm:PinHeader_1x02_P2.54mm_Vertical, F.Cu at (432.5, 254.7)
- added J2004: Conn_01x02_Pin, Connector_PinHeader_2.54mm:PinHeader_1x02_P2.54mm_Vertical, F.Cu at (437.2, 254.7)
- added L11001: 150nH, work:IND_IHVR-4025JZ-3Z_VIS, F.Cu at (397.4, 221.2)
- added L12001: 150nH, work:IND_IHVR-4025JZ-3Z_VIS, F.Cu at (337.9, 221.2)
- added L13001: 150nH, work:IND_IHVR-4025JZ-3Z_VIS, F.Cu at (367.7, 221.2)
- added L14001: 150nH, work:IND_IHVR-4025JZ-3Z_VIS, F.Cu at (367.7, 271.4)
- added L15001: 150nH, work:IND_IHVR-4025JZ-3Z_VIS, F.Cu at (337.9, 246.3)
- added L16002: 150nH, work:IND_IHVR-4025JZ-3Z_VIS, F.Cu at (337.9, 196.1)
- added L17001: 150nH, work:IND_IHVR-4025JZ-3Z_VIS, F.Cu at (397.4, 246.3)
- added L18001: 150nH, work:IND_IHVR-4025JZ-3Z_VIS, F.Cu at (367.7, 196.1)
- added L19001: 150nH, work:IND_IHVR-4025JZ-3Z_VIS, F.Cu at (337.9, 271.4)
- added L3001: 150nH, work:IND_IHVR-4025JZ-3Z_VIS, F.Cu at (397.4, 196.1)
- added L6001: 150nH, work:IND_IHVR-4025JZ-3Z_VIS, F.Cu at (397.4, 271.4)
- added L9001: 150nH, work:IND_IHVR-4025JZ-3Z_VIS, F.Cu at (367.7, 246.3)
- added R11001: 2.2, Resistor_SMD:R_0805_2012Metric, F.Cu at (414.7, 216.8)
- added R11002: 0, Resistor_SMD:R_0805_2012Metric, F.Cu at (414.7, 219.7)
- added R12001: 2.2, Resistor_SMD:R_0805_2012Metric, F.Cu at (355.2, 216.8)
- added R12002: 0, Resistor_SMD:R_0805_2012Metric, F.Cu at (355.2, 219.7)
- added R13001: 2.2, Resistor_SMD:R_0805_2012Metric, F.Cu at (385.0, 216.8)
- added R13002: 0, Resistor_SMD:R_0805_2012Metric, F.Cu at (385.0, 219.7)
- added R14001: 2.2, Resistor_SMD:R_0805_2012Metric, F.Cu at (385.0, 267.0)
- added R14002: 0, Resistor_SMD:R_0805_2012Metric, F.Cu at (385.0, 270.0)
- added R15001: 2.2, Resistor_SMD:R_0805_2012Metric, F.Cu at (355.2, 241.9)
- added R15002: 0, Resistor_SMD:R_0805_2012Metric, F.Cu at (355.2, 244.8)
- added R16003: 2.2, Resistor_SMD:R_0805_2012Metric, F.Cu at (355.2, 191.7)
- added R16004: 0, Resistor_SMD:R_0805_2012Metric, F.Cu at (355.2, 194.6)
- added R17001: 2.2, Resistor_SMD:R_0805_2012Metric, F.Cu at (414.7, 241.9)
- added R17002: 0, Resistor_SMD:R_0805_2012Metric, F.Cu at (414.7, 244.8)
- added R18001: 2.2, Resistor_SMD:R_0805_2012Metric, F.Cu at (385.0, 191.7)
- added R18002: 0, Resistor_SMD:R_0805_2012Metric, F.Cu at (385.0, 194.6)
- added R19001: 2.2, Resistor_SMD:R_0805_2012Metric, F.Cu at (355.2, 267.0)
- added R19002: 0, Resistor_SMD:R_0805_2012Metric, F.Cu at (355.2, 270.0)
- added R3001: 2.2, Resistor_SMD:R_0805_2012Metric, F.Cu at (414.7, 191.7)
- added R3002: 0, Resistor_SMD:R_0805_2012Metric, F.Cu at (414.7, 194.6)
- added R6001: 2.2, Resistor_SMD:R_0805_2012Metric, F.Cu at (414.7, 267.0)
- added R6002: 0, Resistor_SMD:R_0805_2012Metric, F.Cu at (414.7, 270.0)
- added R9001: 2.2, Resistor_SMD:R_0805_2012Metric, F.Cu at (385.0, 241.9)
- added R9002: 0, Resistor_SMD:R_0805_2012Metric, F.Cu at (385.0, 244.8)
- added U11001: AOZ5276QI, work:AOZ5276QI, F.Cu at (415.7, 211.7)
- added U12001: AOZ5276QI, work:AOZ5276QI, F.Cu at (356.2, 211.7)
- added U13001: AOZ5276QI, work:AOZ5276QI, F.Cu at (385.9, 211.7)
- added U14001: AOZ5276QI, work:AOZ5276QI, F.Cu at (385.9, 261.9)
- added U15001: AOZ5276QI, work:AOZ5276QI, F.Cu at (356.2, 236.8)
- added U16002: AOZ5276QI, work:AOZ5276QI, F.Cu at (356.2, 186.6)
- added U17001: AOZ5276QI, work:AOZ5276QI, F.Cu at (415.7, 236.8)
- added U18001: AOZ5276QI, work:AOZ5276QI, F.Cu at (385.9, 186.6)
- added U19001: AOZ5276QI, work:AOZ5276QI, F.Cu at (356.2, 261.9)
- added U2001: TPS536C7B1RSLT, work:QFN48_6X6_TEX, F.Cu at (425.3, 263.9)
- added U3001: AOZ5276QI, work:AOZ5276QI, F.Cu at (415.7, 186.6)
- added U6001: AOZ5276QI, work:AOZ5276QI, F.Cu at (415.7, 261.9)
- added U9001: AOZ5276QI, work:AOZ5276QI, F.Cu at (385.9, 236.8)
- moved C5003 4.35 mm to (180.8, 86.8), turned to -90 degrees
- moved R5005 2.86 mm to (195.9, 78.0)
- moved R5003 2.60 mm to (181.6, 77.4)
- moved TP5006 2.16 mm to (199.7, 77.8)
- moved TP5003 1.92 mm to (178.2, 77.2)
- renumbered C10 to C2001, C4 to C2002, C2 to C2003, C11 to C2004, C1 to C2005, C12 to C2006, C5 to C2007, C3 to C2008, C6 to C2009, C9 to C2010, C7 to C2011, C8 to C2012, R9 to R2001, R10 to R2002, R1 to R2003, R3 to R2004, R11 to R2007, R12 to R2008, R2 to R2010, R4 to R2011, R13 to R2013, R14 to R2014, R15 to R2015, R16 to R2016, R17 to R2017, R18 to R2018, R19 to R2019, R20 to R2020
Connections:
- net /Low Current Supply/+5V  renamed 5V
- net 12V_CUR_SENS renamed /U Controller/PA0
- C2008 pad 1: /VRM Controller/B_TEMP -> MEM_TEMP
- C2009 pad 1: /VRM Controller/A_TEMP -> CORE_TEMO
- C5001 pad 1: /Low Current Supply/12v_spply_lw_crrnt_spply_dcpwr -> 12V
- TP5001 pad 1: /Low Current Supply/12v_spply_lw_crrnt_spply_dcpwr -> 12V
- U5001 pad 2: /Low Current Supply/12v_spply_lw_crrnt_spply_dcpwr -> 12V
- U5001 pad 3: /Low Current Supply/12v_spply_lw_crrnt_spply_dcpwr -> 12V
Routing:
- net Net-(U5001-VOS): track 0.00 -> 40.8 mm
- net GND: track 113.1 -> 128.5 mm, vias 30 -> 40
- net Net-(U5002-OUT): track 0.00 -> 14.6 mm
- net 12V: track 0.00 -> 8.58 mm
- net Net-(U5001-SW): track 0.00 -> 5.54 mm, vias 0 -> 2
- net 3.3V: track 91.6 -> 94.5 mm
- net Net-(D5001-A): track 0.00 -> 2.86 mm
- net 5V: track 0.00 -> 2.79 mm
- net Net-(U5001-PG): track 0.00 -> 2.53 mm
- net Net-(D5002-A): track 0.00 -> 2.16 mm
