File: hardware/U_Controller.kicad_sch (KiCad schematic)
At the start: 22 parts, among them J7002 Conn_ARM_JTAG_SWD_10, J7003 USB_C_Receptacle_USB2.0_16P, SW7001 SW_Wuerth_450301014042, U7001 STM32F401RBTx, U7003 USBLC6-2SC6, Y7001 8Mhz, 16pF

Commit message: chore: DRC violations fixed
Connections:
- net GND: now also J7003.0 (GND), J7003.1 (GND), J7003.2 (GND), J7003.3 (GND)
Changed lines of the file:
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@@
 	)
 	(junction
+		(at 34.29 81.28)
+		(diameter 0)
+		(color 0 0 0 0)
+	)
+	(junction
 		(at 48.26 41.91)
 		(diameter 0)
@@
 	)
 	(junction
-		(at 157.48 22.86)
+		(at 34.29 80.01)
 		(diameter 0)
 		(color 0 0 0 0)
 	)
 	(junction
-		(at 45.72 60.96)
+		(at 157.48 22.86)
 		(diameter 0)
 		(color 0 0 0 0)
 	)
 	(junction
-		(at 26.67 80.01)
+		(at 45.72 60.96)
 		(diameter 0)
 		(color 0 0 0 0)
@@
 	)
 	(junction
+		(at 30.9903 79.9627)
+		(diameter 0)
+		(color 0 0 0 0)
+	)
+	(junction
+		(at 27.0533 79.9627)
+		(diameter 0)
+		(color 0 0 0 0)
+	)
+	(junction
 		(at 46.99 137.16)
 		(diameter 0)
@@
 	)
 	(junction
+		(at 28.9656 79.9627)
+		(diameter 0)
+		(color 0 0 0 0)
+	)
+	(junction
 		(at 156.21 22.86)
 		(diameter 0)
@@
 	(wire
 		(pts
+			(xy 30.9903 79.8877) (xy 30.9903 79.9627)
+		)
+		(stroke
+			(width 0)
+			(type default)
+		)
+	)
+	(wire
+		(pts
 			(xy 127 48.26) (xy 137.16 48.26)
 		)
@@
 	(wire
 		(pts
+			(xy 27.0533 80.0377) (xy 27.0533 79.9627)
+		)
+		(stroke
+			(width 0)
+			(type default)
+		)
+	)
+	(wire
+		(pts
 			(xy 219.71 48.26) (xy 226.06 48.26)
 		)
@@
 	(wire
 		(pts
+			(xy 30.9903 80.01) (xy 34.29 80.01)
+		)
+		(stroke
+			(width 0)
+			(type default)
+		)
+	)
+	(wire
+		(pts
 			(xy 154.94 22.86) (xy 156.21 22.86)
 		)
@@
 	(wire
 		(pts
+			(xy 30.9903 79.9627) (xy 30.9903 80.01)
+		)
+		(stroke
+			(width 0)
+			(type default)
+		)
+	)
+	(wire
+		(pts
 			(xy 25.4 19.05) (xy 33.02 19.05)
 		)
@@
 	(wire
 		(pts
+			(xy 27.0533 79.9627) (xy 28.9656 79.9627)
+		)
+		(stroke
+			(width 0)
+			(type default)
+		)
+	)
+	(wire
+		(pts
 			(xy 48.26 50.8) (xy 46.99 50.8)
 		)
@@
 	(wire
 		(pts
-			(xy 26.67 80.01) (xy 30.48 80.01)
+			(xy 22.86 81.28) (xy 34.29 81.28)
 		)
 		(stroke
@@
 	(wire
 		(pts
+			(xy 24.916 80.0377) (xy 27.0533 80.0377)
+		)
+		(stroke
+			(width 0)
+			(type default)
+		)
+	)
+	(wire
+		(pts
 			(xy 45.72 60.96) (xy 46.99 60.96)
 		)
@@
 	(wire
 		(pts
-			(xy 58.42 142.24) (xy 68.58 142.24)
+			(xy 34.29 81.28) (xy 34.29 80.01)
 		)
 		(stroke
@@
 	(wire
 		(pts
-			(xy 46.99 60.96) (xy 46.99 59.69)
+			(xy 58.42 142.24) (xy 68.58 142.24)
 		)
 		(stroke
@@
 	(wire
 		(pts
-			(xy 172.72 96.52) (xy 179.07 96.52)
+			(xy 46.99 60.96) (xy 46.99 59.69)
 		)
 		(stroke
@@
 	(wire
 		(pts
-			(xy 152.4 22.86) (xy 154.94 22.86)
+			(xy 172.72 96.52) (xy 179.07 96.52)
 		)
 		(stroke
@@
 	(wire
 		(pts
-			(xy 22.86 80.01) (xy 26.67 80.01)
+			(xy 152.4 22.86) (xy 154.94 22.86)
 		)
 		(stroke
@@
 	(wire
 		(pts
+			(xy 22.86 80.01) (xy 22.86 81.28)
+		)
+		(stroke
+			(width 0)
+			(type default)
+		)
+	)
+	(wire
+		(pts
 			(xy 172.72 83.82) (xy 179.07 83.82)
 		)
@@
 	(wire
 		(pts
+			(xy 28.9656 79.9627) (xy 30.9903 79.9627)
+		)
+		(stroke
+			(width 0)
+			(type default)
+		)
+	)
+	(wire
+		(pts
 			(xy 46.99 137.16) (xy 50.8 137.16)
 		)
@@
 	(symbol
 		(lib_id "power:GND")
-		(at 26.67 80.01 0)
+		(at 34.29 81.28 0)
 		(unit 1)
 		(exclude_from_sim no)
@@
 		(on_board yes)
 		(dnp no)
-		(fields_autoplaced yes)
 		(property "Reference" "#PWR07002"
-			(at 26.67 86.36 0)
+			(at 34.29 87.63 0)
 			(effects
 				(font
@@
 		)
 		(property "Value" "GND"
-			(at 26.67 85.09 0)
+			(at 34.29 86.36 0)
 			(effects
 				(font
@@
 		)
 		(property "Footprint" ""
-			(at 26.67 80.01 0)
+			(at 34.29 81.28 0)
 			(effects
 				(font
@@
 		)
 		(property "Datasheet" ""
-			(at 26.67 80.01 0)
+			(at 34.29 81.28 0)
 			(effects
 				(font
@@
 		)
 		(property "Description" "Power symbol creates a global label with name \"GND\" , ground"
-			(at 26.67 80.01 0)
+			(at 34.29 81.28 0)
 			(effects
 				(font
@@
 		(pin "A12"
 		)
+		(pin "0"
+		)
+		(pin "1"
+		)
+		(pin "3"
+		)
+		(pin "2"
+		)
 		(instances

Commit message: feat(pcb): final final final changes
Parts:
- added R7011: 100k, Resistor_SMD:R_0402_1005Metric, symbol Device:R
Connections:
- net +3.3V: now also R7011.1
- net PMBUS_SMBA: now also R7010.1
- net at J7002.2 (SWDIO/TMS), R7004.2, R7006.1: no longer J7002.10 (~{RESET}), R7008.1
- net SMBA renamed I2C_SMBA
- net I2C_SMBA: no longer R7010.1
- new net: J7002.10 (~{RESET}), R7008.1, R7011.2
Changed lines of the file:
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@@
 	)
 	(junction
+		(at 44.45 132.08)
+		(diameter 0)
+		(color 0 0 0 0)
+	)
+	(junction
 		(at 25.4 19.05)
 		(diameter 0)
@@
 	)
 	(junction
-		(at 49.53 132.08)
+		(at 44.45 124.46)
 		(diameter 0)
 		(color 0 0 0 0)
@@
 	(wire
 		(pts
+			(xy 44.45 124.46) (xy 49.53 124.46)
+		)
+		(stroke
+			(width 0)
+			(type default)
+		)
+	)
+	(wire
+		(pts
 			(xy 154.94 22.86) (xy 156.21 22.86)
 		)
@@
 	(wire
 		(pts
+			(xy 44.45 132.08) (xy 50.8 132.08)
+		)
+		(stroke
+			(width 0)
+			(type default)
+		)
+	)
+	(wire
+		(pts
 			(xy 48.26 50.8) (xy 46.99 50.8)
 		)
@@
 	(wire
 		(pts
-			(xy 27.94 124.46) (xy 49.53 124.46)
+			(xy 27.94 124.46) (xy 44.45 124.46)
 		)
 		(stroke
@@
 	(wire
 		(pts
-			(xy 49.53 132.08) (xy 50.8 132.08)
-		)
-		(stroke
-			(width 0)
-			(type default)
-		)
-	)
-	(wire
-		(pts
 			(xy 130.81 73.66) (xy 137.16 73.66)
 		)
@@
 	(wire
 		(pts
-			(xy 40.64 132.08) (xy 49.53 132.08)
+			(xy 40.64 132.08) (xy 44.45 132.08)
 		)
 		(stroke
@@
 		)
 	)
-	(label "SMBA"
-		(at 179.07 53.34 180)
+	(label "I2C_SMBA"
+		(at 179.07 53.34 0)
 		(effects
 			(font
 				(size 1.27 1.27)
 			)
-			(justify right bottom)
+			(justify left bottom)
 		)
 	)
@@
 		)
 	)
-	(label "SMBA"
-		(at 53.34 92.71 0)
-		(effects
-			(font
-				(size 1.27 1.27)
-			)
-			(justify left bottom)
-		)
-	)
 	(label "PB13"
 		(at 179.07 104.14 180)
@@
 		)
 	)
+	(global_label "PMBUS_SMBA"
+		(shape input)
+		(at 53.34 92.71 0)
+		(fields_autoplaced yes)
+		(effects
+			(font
+				(size 1.27 1.27)
+			)
+			(justify left)
+		)
+		(property "Intersheetrefs" "${INTERSHEET_REFS}"
+			(at 68.8437 92.71 0)
+			(effects
+				(font
+					(size 1.27 1.27)
+				)
+				(justify left)
+				(hide yes)
+			)
+		)
+	)
 	(global_label "OB_UP"
 		(shape input)
@@
 					(unit 1)
 				)
+			)
+		)
+	)
+	(symbol
+		(lib_id "Device:R")
+		(at 44.45 128.27 0)
+		(unit 1)
+		(exclude_from_sim no)
+		(in_bom yes)
+		(on_board yes)
+		(dnp no)
+		(property "Reference" "R7011"
+			(at 46.99 129.54 90)
+			(effects
+				(font
+					(size 1.27 1.27)
+				)
+				(justify left)
+			)
+		)
+		(property "Value" "100k"
+			(at 44.45 130.81 90)
+			(effects
+				(font
+					(size 1.27 1.27)
+				)
+				(justify left)
+			)
+		)
+		(property "Footprint" "Resistor_SMD:R_0402_1005Metric"
+			(at 42.672 128.27 90)
+			(effects
+				(font
+					(size 1.27 1.27)
+				)
+				(hide yes)
+			)
+		)
+		(property "Datasheet" "https://jlcpcb.com/partdetail/26484-0402WGF1003TCE/C25741"
+			(at 44.45 128.27 0)
+			(effects
+				(font
+					(size 1.27 1.27)
+				)
+				(hide yes)
+			)
+		)
+		(property "Description" "Resistor"
+			(at 44.45 128.27 0)
+			(effects
+				(font
+					(size 1.27 1.27)
+				)
+				(hide yes)
+			)
+		)
+		(pin "1"
+		)
+		(pin "2"
+		)
+		(instances
+			(project "gpu-external-power-supply"
+				(path "/d5303413-7068-41ba-88e3-39dfa38d31b7/027ff087-ab1d-45e5-9d8f-c94102656fe5"
+					(reference "R7011")
+					(unit 1)
+				)

Commit message: chore(schematic): add LCSC Part Numbers
Parts:
- C7001, C7002: LCSC Part Number (none) -> C1554
- C7003: LCSC Part Number (none) -> C23733
- C7004: LCSC Part Number (none) -> C1581
- D7002: LCSC Part Number (none) -> C2286
- J7002: LCSC Part Number (none) -> C42372555
- J7003: LCSC Part Number (none) -> C2927038
- R7001, R7002: LCSC Part Number (none) -> C25905
- R7003: LCSC Part Number (none) -> C100126
- R7004, R7009, R7011: LCSC Part Number (none) -> C25741
- R7005, R7006, R7007, R7008: LCSC Part Number (none) -> C25076
- R7010: LCSC Part Number (none) -> C17798
- SW7001: LCSC Part Number (none) -> C92658
- U7001: LCSC Part Number (none) -> C75278
- U7003: LCSC Part Number (none) -> C2687116
- Y7001: LCSC Part Number (none) -> C7045397
Changed lines of the file:
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@@
+			)
+		)
+		(property "LCSC Part Number" "C7045397"
+			(at 27.94 102.87 0)
+			(effects
+				(font
+					(size 1.27 1.27)
+				)
+				(hide yes)
 			)
 		)
@@
 		)
 		(property "Description" "Unpolarized capacitor"
+			(at 21.59 96.52 0)
+			(effects
+				(font
+					(size 1.27 1.27)
+				)
+				(hide yes)
+			)
+		)
+		(property "LCSC Part Number" "C1554"
 			(at 21.59 96.52 0)
 			(effects
@@
 			)
 		)
+		(property "LCSC Part Number" "C17798"
+			(at 53.34 96.52 0)
+			(effects
+				(font
+					(size 1.27 1.27)
+				)
+				(hide yes)
+			)
+		)
 		(pin "2"
 		)
@@
 			)
 		)
+		(property "LCSC Part Number" "C25076"
+			(at 54.61 142.24 0)
+			(effects
+				(font
+					(size 1.27 1.27)
+				)
+				(hide yes)
+			)
+		)
 		(pin "1"
 		)
@@
 			)
 		)
+		(property "LCSC Part Number" ""
+			(at 245.11 25.4 0)
+			(effects
+				(font
+					(size 1.27 1.27)
+				)
+				(hide yes)
+			)
+		)
 		(pin "1"
 		)
@@
 			)
 		)
+		(property "LCSC Part Number" "C25076"
+			(at 54.61 137.16 0)
+			(effects
+				(font
+					(size 1.27 1.27)
+				)
+				(hide yes)
+			)
+		)
 		(pin "1"
 		)
@@
 		)
 		(property "Description" "Unpolarized capacitor"
+			(at 25.4 22.86 0)
+			(effects
+				(font
+					(size 1.27 1.27)
+				)
+				(hide yes)
+			)
+		)
+		(property "LCSC Part Number" "C23733"
 			(at 25.4 22.86 0)
 			(effects
@@
 			)
 		)
+		(property "LCSC Part Number" "C25076"
+			(at 54.61 139.7 0)
+			(effects
+				(font
+					(size 1.27 1.27)
+				)
+				(hide yes)
+			)
+		)
 		(pin "1"
 		)
@@
 		)
 		(property "Description" "Unpolarized capacitor"
+			(at 21.59 110.49 0)
+			(effects
+				(font
+					(size 1.27 1.27)
+				)
+				(hide yes)
+			)
+		)
+		(property "LCSC Part Number" "C1554"
 			(at 21.59 110.49 0)
 			(effects
@@
 			)
 		)
+		(property "LCSC Part Number" "C92658"
+			(at 256.54 21.59 0)
+			(effects
+				(font
+					(size 1.27 1.27)
+				)
+				(hide yes)
+			)
+		)
 		(pin "2"
 		)
@@
 			)
 		)
+		(property "LCSC Part Number" "C100126"
+			(at 233.68 25.4 0)
+			(effects
+				(font
+					(size 1.27 1.27)
+				)
+				(hide yes)
+			)
+		)
 		(pin "2"
 		)
@@
 			)
 		)
+		(property "LCSC Part Number" "C25741"
+			(at 46.99 147.32 0)
+			(effects
+				(font
+					(size 1.27 1.27)
+				)
+				(hide yes)
+			)
+		)
 		(pin "1"
 		)
@@
 			)
 		)
+		(property "LCSC Part Number" "C1581"
+			(at 33.02 22.86 0)
+			(effects
+				(font
+					(size 1.27 1.27)
+				)
+				(hide yes)
+			)
+		)
 		(pin "2"
 		)
@@
 		)
 		(property "Description" "Resistor"
+			(at 52.07 50.8 0)
+			(effects
+				(font
+					(size 1.27 1.27)
+				)
+				(hide yes)
+			)
+		)
+		(property "LCSC Part Number" "C25905"
 			(at 52.07 50.8 0)
 			(effects
@@
 			)
 		)
+		(property "LCSC Part Number" "C75278"
+			(at 154.94 71.12 0)
+			(effects
+				(font
+					(size 1.27 1.27)
+				)
+				(hide yes)
+			)
+		)
 		(pin "63"
 		)
@@
 			)
 		)
+		(property "LCSC Part Number" "C2286"
+			(at 53.34 104.14 0)
+			(effects
+				(font
+					(size 1.27 1.27)
+				)
+				(hide yes)
+			)
+		)
 		(pin "2"
 		)
@@
 			)
 		)
+		(property "LCSC Part Number" "C25905"
+			(at 52.07 45.72 0)
+			(effects
+				(font
+					(size 1.27 1.27)
+				)
+				(hide yes)
+			)
+		)
 		(pin "2"
 		)
@@
 		)
 		(property "Description" "Very low capacitance ESD protection diode, 2 data-line, SOT-23-6"
+			(at 57.15 57.15 0)
+			(effects
+				(font
+					(size 1.27 1.27)
+				)
+				(hide yes)
+			)
+		)
+		(property "LCSC Part Number" "C2687116"
 			(at 57.15 57.15 0)
 			(effects
@@
 			)
 		)
+		(property "LCSC Part Number" "C25076"
+			(at 54.61 132.08 0)
+			(effects
+				(font
+					(size 1.27 1.27)
+				)
+				(hide yes)
+			)
+		)
 		(pin "1"
 		)
@@
 			)
 		)
+		(property "LCSC Part Number" "C2927038"
+			(at 30.48 57.15 0)
+			(effects
+				(font
+					(size 1.27 1.27)
+				)
+				(hide yes)
+			)
+		)
 		(pin "B8"
 		)
@@
 			)
 		)
+		(property "LCSC Part Number" "C25741"
+			(at 44.45 128.27 0)
+			(effects
+				(font
+					(size 1.27 1.27)
+				)
+				(hide yes)
+			)
+		)
 		(pin "1"
 		)
@@
 			)
 		)
+		(property "LCSC Part Number" "C42372555"
+			(at 27.94 139.7 0)
+			(effects
+				(font
+					(size 1.27 1.27)
+				)
+				(hide yes)
+			)
+		)
 		(pin "8"
 		)
@@
 			(at 49.53 128.27 0)
 			(effects
+				(font
+					(size 1.27 1.27)
+				)
+				(hide yes)
+			)
+		)
+		(property "LCSC Part Number" "C25741"
+			(at 49.53 128.27 0)
+			(effects
