File: hardware/Vcore_Stage.kicad_sch (KiCad schematic)
At the start: 21 parts, among them U16002 AOZ5276QI

Commit message: feat(schematic): added cooler mounting holes
added cooler mounting holes to schematic
changed temp pins to read proper tempurature
small fixes
Parts:
- removed C16022: 47pF, Capacitor_SMD:C_0805_2012Metric, symbol Device:C
- C16018, C16019, C16020, C16021, C16023, C16024, C16032, C16033, C16034: footprint Capacitor_SMD:C_0805_2012Metric -> Capacitor_SMD:C_0402_1005Metric
- C16027: value 22uF -> 47uF; footprint Capacitor_SMD:C_0805_2012Metric -> Capacitor_SMD:C_1210_3225Metric
- C16028, C16031: footprint Capacitor_THT:CP_Radial_D6.3mm_P2.50mm -> Capacitor_SMD:CP_Elec_6.3x7.7
- R16003, R16004: footprint Resistor_SMD:R_0805_2012Metric -> Resistor_SMD:R_0402_1005Metric
Changed lines of the file:
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@@
 	)
 	(junction
-		(at 135.89 97.79)
-		(diameter 0)
-		(color 0 0 0 0)
-	)
-	(junction
 		(at 238.76 72.39)
 		(diameter 0)
@@
 	)
 	(junction
-		(at 129.54 113.03)
-		(diameter 0)
-		(color 0 0 0 0)
-	)
-	(junction
 		(at 114.3 62.23)
 		(diameter 0)
@@
 	(wire
 		(pts
-			(xy 124.46 97.79) (xy 135.89 97.79)
+			(xy 124.46 97.79) (xy 140.97 97.79)
 		)
 		(stroke
@@
 	(wire
 		(pts
-			(xy 135.89 113.03) (xy 129.54 113.03)
-		)
-		(stroke
-			(width 0)
-			(type default)
-		)
-	)
-	(wire
-		(pts
-			(xy 135.89 101.6) (xy 135.89 97.79)
-		)
-		(stroke
-			(width 0)
-			(type default)
-		)
-	)
-	(wire
-		(pts
 			(xy 118.11 105.41) (xy 121.92 105.41)
 		)
@@
 	(wire
 		(pts
-			(xy 135.89 109.22) (xy 135.89 113.03)
-		)
-		(stroke
-			(width 0)
-			(type default)
-		)
-	)
-	(wire
-		(pts
 			(xy 208.28 95.25) (xy 196.85 95.25)
 		)
@@
 	(wire
 		(pts
-			(xy 135.89 97.79) (xy 140.97 97.79)
-		)
-		(stroke
-			(width 0)
-			(type default)
-		)
-	)
-	(wire
-		(pts
 			(xy 140.97 86.36) (xy 140.97 87.63)
 		)
@@
 			)
 		)
-		(property "Footprint" "Capacitor_SMD:C_0805_2012Metric"
+		(property "Footprint" "Capacitor_SMD:C_0402_1005Metric"
 			(at 166.0652 104.14 0)
 			(effects
@@
 			)
 		)
-		(property "Datasheet" "~"
+		(property "Datasheet" "https://jlcpcb.com/partdetail/1933-0402F104M500NT/C1581"
 			(at 165.1 100.33 0)
 			(effects
@@
 			)
 		)
-		(property "Footprint" "Capacitor_SMD:C_0805_2012Metric"
+		(property "Footprint" "Capacitor_SMD:C_0402_1005Metric"
 			(at 228.2952 80.01 0)
 			(effects
@@
 			)
 		)
-		(property "Datasheet" "~"
+		(property "Datasheet" "https://jlcpcb.com/partdetail/24469-CL05A475MP5NRNC/C23733"
 			(at 227.33 76.2 0)
 			(effects
@@
 			)
 		)
-		(property "Datasheet" "~"
+		(property "Datasheet" "https://jlcpcb.com/partdetail/46786-CL21A226MAQNNNE/C45783"
 			(at 175.26 100.33 0)
 			(effects
@@
 			)
 		)
-		(property "Footprint" "Capacitor_SMD:C_0805_2012Metric"
+		(property "Footprint" "Capacitor_SMD:C_0402_1005Metric"
 			(at 115.2652 72.39 0)
 			(effects
@@
 			)
 		)
-		(property "Datasheet" "~"
+		(property "Datasheet" "https://jlcpcb.com/partdetail/13164-CL05A225MQ5NSNC/C12530"
 			(at 114.3 68.58 0)
 			(effects
@@
 			)
 		)
-		(property "Footprint" "Resistor_SMD:R_0805_2012Metric"
+		(property "Footprint" "Resistor_SMD:R_0402_1005Metric"
 			(at 121.92 61.468 90)
 			(effects
@@
 			)
 		)
-		(property "Datasheet" "~"
+		(property "Datasheet" "https://jlcpcb.com/partdetail/25901-0402WGJ022JTCE/C25158"
 			(at 121.92 59.69 0)
 			(effects
@@
 			)
 		)
-		(property "Footprint" "Resistor_SMD:R_0805_2012Metric"
+		(property "Footprint" "Resistor_SMD:R_0402_1005Metric"
 			(at 127 88.138 90)
 			(effects
@@
 			)
 		)
-		(property "Datasheet" "~"
+		(property "Datasheet" "https://jlcpcb.com/partdetail/17853-0402WGF0000TCE/C17168"
 			(at 127 86.36 0)
 			(effects
@@
 			)
 		)
-		(property "Datasheet" "https://www.digikey.com/en/products/detail/panasonic-electronic-components/EEF-SX0D471XE/1731681"
+		(property "Datasheet" "https://jlcpcb.com/partdetail/Panasonic-EEFGX0E471R/C139572"
 			(at 179.07 76.2 0)
 			(effects
@@
 			)
 		)
-		(property "Datasheet" "~"
+		(property "Datasheet" "https://jlcpcb.com/partdetail/46786-CL21A226MAQNNNE/C45783"
 			(at 196.85 100.33 0)
 			(effects
@@
 			)
 		)
-		(property "Value" "22uF"
+		(property "Value" "47uF"
 			(at 189.23 101.5999 0)
 			(effects
@@
 			)
 		)
-		(property "Footprint" "Capacitor_SMD:C_0805_2012Metric"
+		(property "Footprint" "Capacitor_SMD:C_1210_3225Metric"
 			(at 186.3852 104.14 0)
 			(effects
@@
 			)
 		)
-		(property "Datasheet" "~"
+		(property "Datasheet" "https://jlcpcb.com/partdetail/MurataElectronics-GRM32ER61C476KE15L/C77101"
 			(at 185.42 100.33 0)
 			(effects
@@
 	(symbol
 		(lib_id "Device:C")
-		(at 135.89 105.41 0)
-		(unit 1)
-		(exclude_from_sim no)
-		(in_bom yes)
-		(on_board yes)
-		(dnp no)
-		(property "Reference" "C16022"
-			(at 129.794 101.346 0)
-			(effects
-				(font
-					(size 1.27 1.27)
-				)
-				(justify left)
-			)
-		)
-		(property "Value" "47pF"
-			(at 129.794 103.886 0)
-			(effects
-				(font
-					(size 1.27 1.27)
-				)
-				(justify left)
-			)
-		)
-		(property "Footprint" "Capacitor_SMD:C_0805_2012Metric"
-			(at 136.8552 109.22 0)
-			(effects
-				(font
-					(size 1.27 1.27)
-				)
-				(hide yes)
-			)
-		)
-		(property "Datasheet" "~"
-			(at 135.89 105.41 0)
-			(effects
-				(font
-					(size 1.27 1.27)
-				)
-				(hide yes)
-			)
-		)
-		(property "Description" "Unpolarized capacitor"
-			(at 135.89 105.41 0)
-			(effects
-				(font
-					(size 1.27 1.27)
-				)
-				(hide yes)
-			)
-		)
-		(pin "2"
-		)
-		(pin "1"
-		)
-		(instances
-			(project "gpu-external-power-supply"
-				(path "/d5303413-7068-41ba-88e3-39dfa38d31b7/49a17099-106d-4abb-ae14-dd757ef91d45"
-					(reference "C16022")
-					(unit 1)
-				)
-				(path "/d5303413-7068-41ba-88e3-39dfa38d31b7/61a0cb7a-9d01-4760-8ce8-789a6ab49ba4"
-					(reference "C12005")
-					(unit 1)
-				)
-				(path "/d5303413-7068-41ba-88e3-39dfa38d31b7/655b25ca-de6c-4e3a-af15-4fcc6e2bd037"
-					(reference "C15005")
-					(unit 1)
-				)
-				(path "/d5303413-7068-41ba-88e3-39dfa38d31b7/69405101-d09e-4d45-aab1-12aa0a1b3acb"
-					(reference "C19005")
-					(unit 1)
-				)
-				(path "/d5303413-7068-41ba-88e3-39dfa38d31b7/6b7e5349-9b9f-40b8-b2bb-5c34bbc51f14"
-					(reference "C18005")
-					(unit 1)
-				)
-				(path "/d5303413-7068-41ba-88e3-39dfa38d31b7/95d79d2d-f5ad-46ce-832a-3e27966061c2"
-					(reference "C13005")
-					(unit 1)
-				)
-				(path "/d5303413-7068-41ba-88e3-39dfa38d31b7/c5652880-1b75-42d4-a1cb-09cfb95d4a18"
-					(reference "C14005")
-					(unit 1)
-				)
-				(path "/d5303413-7068-41ba-88e3-39dfa38d31b7/d8c0ae4b-1079-42a5-9412-f5c12c8efe93"
-					(reference "C11005")
-					(unit 1)
-				)
-				(path "/d5303413-7068-41ba-88e3-39dfa38d31b7/d9fa39fa-1ff5-40d0-a988-b7fa258daa9e"
-					(reference "C17005")
-					(unit 1)
-				)
-				(path "/d5303413-7068-41ba-88e3-39dfa38d31b7/f474b2ec-e107-43c1-9cef-22ba90148aa8"
-					(reference "C6005")
-					(unit 1)
-				)
-			)
-		)
-	)
-	(symbol
-		(lib_id "Device:C")
 		(at 101.6 106.68 0)
 		(unit 1)
@@
 			)
 		)
-		(property "Footprint" "Capacitor_SMD:C_0805_2012Metric"
+		(property "Footprint" "Capacitor_SMD:C_0402_1005Metric"
 			(at 102.5652 110.49 0)
 			(effects
@@
 			)
 		)
-		(property "Datasheet" "~"
+		(property "Datasheet" "https://jlcpcb.com/partdetail/1919-0402CG470J500NT/C1567"
 			(at 101.6 106.68 0)
 			(effects
@@
 			)
 		)
-		(property "Footprint" "Capacitor_THT:CP_Radial_D6.3mm_P2.50mm"
+		(property "Footprint" "Capacitor_SMD:CP_Elec_6.3x7.7"
 			(at 191.4652 80.01 0)
 			(effects
@@
 			)
 		)
-		(property "Datasheet" "https://www.digikey.com/en/products/detail/kyocera-avx/RPA0608221M016B/17634426"
+		(property "Datasheet" "https://jlcpcb.com/partdetail/HonorElec-RVT1C221M0607/C3342"
 			(at 190.5 76.2 0)
 			(effects
@@
 			)
 		)
-		(property "Footprint" "Capacitor_SMD:C_0805_2012Metric"
+		(property "Footprint" "Capacitor_SMD:C_0402_1005Metric"
 			(at 140.97 85.3948 0)
 			(effects
@@
 			)
 		)
-		(property "Datasheet" "~"
+		(property "Datasheet" "https://jlcpcb.com/partdetail/1933-0402F104M500NT/C1581"
 			(at 137.16 86.36 0)
 			(effects
@@
 			)
 		)
-		(property "Datasheet" "~"
+		(property "Datasheet" "https://jlcpcb.com/partdetail/17464-CL21A476MQYNNNE/C16780"
 			(at 201.93 76.2 0)
 			(effects
@@
 			)
 		)
-		(property "Footprint" "Capacitor_SMD:C_0805_2012Metric"
+		(property "Footprint" "Capacitor_SMD:C_0402_1005Metric"
 			(at 126.6952 113.03 0)
 			(effects
@@
 			)
 		)
-		(property "Datasheet" "~"
+		(property "Datasheet" "https://jlcpcb.com/partdetail/1933-0402F104M500NT/C1581"
 			(at 125.73 109.22 0)
 			(effects
@@
 			)
 		)
-		(property "Footprint" "Capacitor_SMD:C_0805_2012Metric"
+		(property "Footprint" "Capacitor_SMD:C_0402_1005Metric"
 			(at 131.7752 73.66 0)
 			(effects
@@
 			)
 		)
-		(property "Datasheet" "~"
+		(property "Datasheet" "https://jlcpcb.com/partdetail/13164-CL05A225MQ5NSNC/C12530"
 			(at 130.81 69.85 0)
 			(effects
@@
 			)
 		)
-		(property "Footprint" "Capacitor_SMD:C_0805_2012Metric"
+		(property "Footprint" "Capacitor_SMD:C_0402_1005Metric"
 			(at 216.8652 80.01 0)
 			(effects
@@
 			)
 		)
-		(property "Datasheet" "~"
+		(property "Datasheet" "https://jlcpcb.com/partdetail/Chinocera-HGC0402R5226M6R3NTEJ/C7432764"
 			(at 215.9 76.2 0)
 			(effects
@@
 			)
 		)
-		(property "Footprint" "Capacitor_THT:CP_Radial_D6.3mm_P2.50mm"
+		(property "Footprint" "Capacitor_SMD:CP_Elec_6.3x7.7"
 			(at 209.2452 104.14 0)
 			(effects
@@
 			)
 		)
-		(property "Datasheet" "https://www.digikey.com/en/products/detail/kyocera-avx/RPA0608221M016B/17634426"
+		(property "Datasheet" "https://jlcpcb.com/partdetail/HonorElec-RVT1C221M0607/C3342"
 			(at 208.28 100.33 0)
 			(effects
@@
 			)
 		)
-		(property "Footprint" "Capacitor_SMD:C_0805_2012Metric"
+		(property "Footprint" "Capacitor_SMD:C_0402_1005Metric"
 			(at 239.7252 80.01 0)
 			(effects
@@
 			)
 		)
-		(property "Datasheet" "~"
+		(property "Datasheet" "https://jlcpcb.com/partdetail/1933-0402F104M500NT/C1581"
 			(at 238.76 76.2 0)
 			(effects

Commit message: chore(schematic): add LCSC Part Numbers
Parts:
- C16018: LCSC Part Number (none) -> C1567
- C16019, C16021: LCSC Part Number (none) -> C12530
- C16020, C16023, C16024, C16034: LCSC Part Number (none) -> C1581
- C16025, C16029: LCSC Part Number (none) -> C45783
- C16026: LCSC Part Number (none) -> C139572
- C16027: LCSC Part Number (none) -> C77101
- C16028, C16031: LCSC Part Number (none) -> C3342
- C16030: LCSC Part Number (none) -> C16780
- C16032: LCSC Part Number (none) -> C7432764
- C16033: LCSC Part Number (none) -> C23733
- L16002: LCSC Part Number (none) -> C19483954
- R16003: LCSC Part Number (none) -> C25158
- R16004: LCSC Part Number (none) -> C17168
- U16002: LCSC Part Number (none) -> C5587859
Changed lines of the file:
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@@
+			)
+		)
+		(property "LCSC Part Number" "C1581"
+			(at 165.1 100.33 0)
+			(effects
+				(font
+					(size 1.27 1.27)
+				)
+				(hide yes)
 			)
 		)
@@
 			)
 		)
+		(property "LCSC Part Number" "C23733"
+			(at 227.33 76.2 0)
+			(effects
+				(font
+					(size 1.27 1.27)
+				)
+				(hide yes)
+			)
+		)
 		(pin "2"
 		)
@@
 			)
 		)
+		(property "LCSC Part Number" "C45783"
+			(at 175.26 100.33 0)
+			(effects
+				(font
+					(size 1.27 1.27)
+				)
+				(hide yes)
+			)
+		)
 		(pin "1"
 		)
@@
 		)
 		(property "Description" "Unpolarized capacitor"
+			(at 114.3 68.58 0)
+			(effects
+				(font
+					(size 1.27 1.27)
+				)
+				(hide yes)
+			)
+		)
+		(property "LCSC Part Number" "C12530"
 			(at 114.3 68.58 0)
 			(effects
@@
 			)
 		)
+		(property "LCSC Part Number" "C25158"
+			(at 121.92 59.69 0)
+			(effects
+				(font
+					(size 1.27 1.27)
+				)
+				(hide yes)
+			)
+		)
 		(pin "2"
 		)
@@
 		)
 		(property "Description" "Resistor"
+			(at 127 86.36 0)
+			(effects
+				(font
+					(size 1.27 1.27)
+				)
+				(hide yes)
+			)
+		)
+		(property "LCSC Part Number" "C17168"
 			(at 127 86.36 0)
 			(effects
@@
 			)
 		)
+		(property "LCSC Part Number" "C139572"
+			(at 179.07 76.2 0)
+			(effects
+				(font
+					(size 1.27 1.27)
+				)
+				(hide yes)
+			)
+		)
 		(pin "2"
 		)
@@
 			)
 		)
+		(property "LCSC Part Number" "C45783"
+			(at 196.85 100.33 0)
+			(effects
+				(font
+					(size 1.27 1.27)
+				)
+				(hide yes)
+			)
+		)
 		(pin "1"
 		)
@@
 			)
 		)
+		(property "LCSC Part Number" "C77101"
+			(at 185.42 100.33 0)
+			(effects
+				(font
+					(size 1.27 1.27)
+				)
+				(hide yes)
+			)
+		)
 		(pin "2"
 		)
@@
 			)
 		)
+		(property "LCSC Part Number" "C1567"
+			(at 101.6 106.68 0)
+			(effects
+				(font
+					(size 1.27 1.27)
+				)
+				(hide yes)
+			)
+		)
 		(pin "1"
 		)
@@
 			)
 		)
+		(property "LCSC Part Number" "C3342"
+			(at 190.5 76.2 0)
+			(effects
+				(font
+					(size 1.27 1.27)
+				)
+				(hide yes)
+			)
+		)
 		(pin "1"
 		)
@@
 		)
 		(property "Description" "Unpolarized capacitor"
+			(at 137.16 86.36 0)
+			(effects
+				(font
+					(size 1.27 1.27)
+				)
+				(hide yes)
+			)
+		)
+		(property "LCSC Part Number" "C1581"
 			(at 137.16 86.36 0)
 			(effects
@@
 			)
 		)
+		(property "LCSC Part Number" "C16780"
+			(at 201.93 76.2 0)
+			(effects
+				(font
+					(size 1.27 1.27)
+				)
+				(hide yes)
+			)
+		)
 		(pin "1"
 		)
@@
 			)
 		)
+		(property "LCSC Part Number" "C1581"
+			(at 125.73 109.22 0)
+			(effects
+				(font
+					(size 1.27 1.27)
+				)
+				(hide yes)
+			)
+		)
 		(pin "1"
 		)
@@
 			)
 		)
+		(property "LCSC Part Number" "C12530"
+			(at 130.81 69.85 0)
+			(effects
+				(font
+					(size 1.27 1.27)
+				)
+				(hide yes)
+			)
+		)
 		(pin "1"
 		)
@@
 			)
 		)
+		(property "LCSC Part Number" "C7432764"
+			(at 215.9 76.2 0)
+			(effects
+				(font
+					(size 1.27 1.27)
+				)
+				(hide yes)
+			)
+		)
 		(pin "1"
 		)
@@
 			)
 		)
+		(property "LCSC Part Number" "C3342"
+			(at 208.28 100.33 0)
+			(effects
+				(font
+					(size 1.27 1.27)
+				)
+				(hide yes)
+			)
+		)
 		(pin "2"
 		)
@@
 			)
 		)
+		(property "LCSC Part Number" "C5587859"
+			(at 149.86 80.01 0)
+			(effects
+				(font
+					(size 1.27 1.27)
+				)
+				(hide yes)
+			)
+		)
 		(pin "36"
 		)
@@
 			)
 		)
+		(property "LCSC Part Number" "C1581"
+			(at 238.76 76.2 0)
+			(effects
+				(font
+					(size 1.27 1.27)
+				)
+				(hide yes)
+			)
+		)
 		(pin "2"
 		)
@@
 			(at 172.72 72.39 0)
 			(effects
+				(font
+					(size 1.27 1.27)
+				)
+				(hide yes)
+			)
+		)
+		(property "LCSC Part Number" "C19483954"
+			(at 172.72 72.39 0)
+			(effects
